File: Onboarding/Michael_Samson_Onboarding/Michael_Samson_Onboarding.kicad_pcb (KiCad board)
At the start: 2 copper layers, 6 parts, among them U2 NE555P

Commit message: msamson
Parts:
- removed R1, R2: Ra, Resistor_SMD:R_1206_3216Metric
- removed R3: R_Small_US, Resistor_SMD:R_1206_3216Metric
- added RA1: 5 kΩ, Resistor_SMD:R_1206_3216Metric, F.Cu at (229.0, 59.5)
- added RB1: 3 kΩ, Resistor_SMD:R_1206_3216Metric, F.Cu at (229.0, 51.0)
- added RL1: 1 kΩ, Resistor_SMD:R_1206_3216Metric, F.Cu at (250.8, 35.7)
- C2: value C_Small_US -> 0.15 µF
- moved U2 38.9 mm to (238.0, 52.9)
- moved C1 34.4 mm to (254.5, 60.0)
- moved C2 21.6 mm to (253.3, 43.2), turned to 180 degrees
