File: Onboarding/Michael_Samson_Onboarding/Michael_Samson_Onboarding.kicad_sch (KiCad schematic)
At the start: 6 parts, among them U2 NE555P

Commit message: Michael Samson onboarding
Parts:
- C1, C2: footprint (none) -> Capacitor_SMD:C_1206_3216Metric
- R1: value Rb -> Ra; footprint (none) -> Resistor_SMD:R_1206_3216Metric
- R2, R3: footprint (none) -> Resistor_SMD:R_1206_3216Metric
Connections:
- no-connect marks 2 -> 1
Changed lines of the file:
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@@
 	(paper "A4")
+	(junction
+		(at 240.03 60.96)
+		(diameter 0)
+		(color 0 0 0 0)
+	)
+	(junction
+		(at 242.57 29.21)
+		(diameter 0)
+		(color 0 0 0 0)
+	)
+	(junction
+		(at 227.33 29.21)
+		(diameter 0)
+		(color 0 0 0 0)
+	)
+	(junction
+		(at 234.95 29.21)
+		(diameter 0)
+		(color 0 0 0 0)
+	)
+	(junction
+		(at 242.57 35.56)
+		(diameter 0)
+		(color 0 0 0 0)
+	)
+	(junction
+		(at 227.33 55.88)
+		(diameter 0)
+		(color 0 0 0 0)
+	)
+	(junction
+		(at 220.98 48.26)
+		(diameter 0)
+		(color 0 0 0 0)
+	)
 	(junction
 		(at 220.98 55.88)
@@
 	)
 	(junction
-		(at 242.57 29.21)
-		(diameter 0)
-		(color 0 0 0 0)
-	)
-	(junction
-		(at 227.33 29.21)
-		(diameter 0)
-		(color 0 0 0 0)
-	)
-	(junction
-		(at 234.95 29.21)
-		(diameter 0)
-		(color 0 0 0 0)
-	)
-	(junction
-		(at 242.57 35.56)
-		(diameter 0)
-		(color 0 0 0 0)
-	)
-	(junction
-		(at 227.33 55.88)
-		(diameter 0)
-		(color 0 0 0 0)
-	)
-	(junction
-		(at 220.98 48.26)
-		(diameter 0)
-		(color 0 0 0 0)
-	)
-	(junction
 		(at 252.73 50.8)
 		(diameter 0)
@@
 	)
 	(no_connect
-		(at 210.82 34.29)
-	)
-	(no_connect
 		(at 240.03 40.64)
 	)
@@
 	(wire
 		(pts
-			(xy 220.98 48.26) (xy 220.98 50.8)
-		)
-		(stroke
-			(width 0)
-			(type default)
-		)
-	)
-	(wire
-		(pts
 			(xy 220.98 41.91) (xy 220.98 48.26)
 		)
@@
 	(wire
 		(pts
+			(xy 220.98 48.26) (xy 220.98 49.53)
+		)
+		(stroke
+			(width 0)
+			(type default)
+		)
+	)
+	(wire
+		(pts
 			(xy 227.33 45.72) (xy 227.33 29.21)
 		)
@@
 		(pts
 			(xy 227.33 29.21) (xy 234.95 29.21)
+		)
+		(stroke
+			(width 0)
+			(type default)
+		)
+	)
+	(wire
+		(pts
+			(xy 220.98 54.61) (xy 220.98 55.88)
 		)
 		(stroke
@@
 		(in_pos_files yes)
 		(dnp no)
-		(fields_autoplaced yes)
 		(property "Reference" "U2"
-			(at 253.365 44.3798 0)
+			(at 250.19 44.45 0)
 			(show_name no)
 			(do_not_autoplace no)
@@
 		)
 		(property "Value" "NE555P"
-			(at 253.365 46.9198 0)
+			(at 247.65 41.91 0)
 			(show_name no)
 			(do_not_autoplace no)
@@
 	)
 	(symbol
-		(lib_id "Device:R_Small_US")
-		(at 220.98 53.34 0)
+		(lib_id "power:PWR_FLAG")
+		(at 240.03 60.96 90)
 		(unit 1)
 		(body_style 1)
@@
 		(in_pos_files yes)
 		(dnp no)
-		(property "Reference" "R1"
-			(at 215.265 52.07 0)
+		(fields_autoplaced yes)
+		(property "Reference" "#FLG02"
+			(at 238.125 60.96 0)
+			(hide yes)
+			(show_name no)
+			(do_not_autoplace no)
+			(effects
+				(font
+					(size 1.27 1.27)
+				)
+			)
+		)
+		(property "Value" "PWR_FLAG"
+			(at 236.22 60.9599 90)
 			(show_name no)
 			(do_not_autoplace no)
@@
 			)
 		)
-		(property "Value" "Rb"
-			(at 215.265 54.61 0)
-			(show_name no)
-			(do_not_autoplace no)
-			(effects
-				(font
-					(size 1.27 1.27)
-				)
-				(justify left)
-			)
-		)
 		(property "Footprint" ""
-			(at 220.98 53.34 0)
+			(at 240.03 60.96 0)
 			(hide yes)
 			(show_name no)
@@
 		)
 		(property "Datasheet" ""
-			(at 220.98 53.34 0)
-			(hide yes)
-			(show_name no)
-			(do_not_autoplace no)
-			(effects
-				(font
-					(size 1.27 1.27)
-				)
-			)
-		)
-		(property "Description" "Resistor, small US symbol"
-			(at 220.98 53.34 0)
-			(hide yes)
-			(show_name no)
-			(do_not_autoplace no)
-			(effects
-				(font
-					(size 1.27 1.27)
-				)
-			)
-		)
-		(pin "2"
+			(at 240.03 60.96 0)
+			(hide yes)
+			(show_name no)
+			(do_not_autoplace no)
+			(effects
+				(font
+					(size 1.27 1.27)
+				)
+			)
+		)
+		(property "Description" "Special symbol for telling ERC where power comes from"
+			(at 240.03 60.96 0)
+			(hide yes)
+			(show_name no)
+			(do_not_autoplace no)
+			(effects
+				(font
+					(size 1.27 1.27)
+				)
+			)
 		)
 		(pin "1"
@@
 			(project "Michael_Samson_Onboarding"
 				(path "/e5003549-9df7-4e7c-9d3a-2812ef50da89"
-					(reference "R1")
+					(reference "#FLG02")
 					(unit 1)
 				)
@@
 			)
 		)
-		(property "Footprint" ""
+		(property "Footprint" "Resistor_SMD:R_1206_3216Metric"
 			(at 220.98 39.37 0)
 			(hide yes)
@@
 			)
 		)
-		(property "Footprint" ""
+		(property "Footprint" "Capacitor_SMD:C_1206_3216Metric"
 			(at 220.98 58.42 0)
 			(hide yes)
@@
 			)
 		)
-		(property "Footprint" ""
+		(property "Footprint" "Capacitor_SMD:C_1206_3216Metric"
 			(at 234.95 31.75 0)
 			(hide yes)
@@
 	)
 	(symbol
+		(lib_id "Device:R_Small_US")
+		(at 220.98 52.07 0)
+		(unit 1)
+		(body_style 1)
+		(exclude_from_sim no)
+		(in_bom yes)
+		(on_board yes)
+		(in_pos_files yes)
+		(dnp no)
+		(property "Reference" "R1"
+			(at 215.9 50.8 0)
+			(show_name no)
+			(do_not_autoplace no)
+			(effects
+				(font
+					(size 1.27 1.27)
+				)
+				(justify left)
+			)
+		)
+		(property "Value" "Ra"
+			(at 215.9 53.34 0)
+			(show_name no)
+			(do_not_autoplace no)
+			(effects
+				(font
+					(size 1.27 1.27)
+				)
+				(justify left)
+			)
+		)
+		(property "Footprint" "Resistor_SMD:R_1206_3216Metric"
+			(at 220.98 52.07 0)
+			(hide yes)
+			(show_name no)
+			(do_not_autoplace no)
+			(effects
+				(font
+					(size 1.27 1.27)
+				)
+			)
+		)
+		(property "Datasheet" ""
+			(at 220.98 52.07 0)
+			(hide yes)
+			(show_name no)
+			(do_not_autoplace no)
+			(effects
+				(font
+					(size 1.27 1.27)
+				)
+			)
+		)
+		(property "Description" "Resistor, small US symbol"
+			(at 220.98 52.07 0)
+			(hide yes)
+			(show_name no)
+			(do_not_autoplace no)
+			(effects
+				(font
+					(size 1.27 1.27)
+				)
+			)
+		)
+		(pin "1"
+		)
+		(pin "2"
+		)
+		(instances
+			(project "Michael_Samson_Onboarding"
+				(path "/e5003549-9df7-4e7c-9d3a-2812ef50da89"
+					(reference "R1")
+					(unit 1)
+				)
+			)
+		)
+	)
+	(symbol
 		(lib_id "power:GND")
 		(at 234.95 34.29 0)
@@
 			)
 		)
-		(property "Footprint" ""
+		(property "Footprint" "Resistor_SMD:R_1206_3216Metric"
 			(at 252.73 39.37 0)
 			(hide yes)

Commit message: msamson
Parts:
- C2: value C_Small_US -> 0.15 µF
- RA1: renamed from R2; value Ra -> 5 kΩ
- RB1: renamed from R1; value Ra -> 3 kΩ
- RL1: renamed from R3; value R_Small_US -> 1 kΩ
Changed lines of the file:
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@@
 		(in_pos_files yes)
 		(dnp no)
-		(property "Reference" "R2"
+		(property "Reference" "RA1"
 			(at 214.63 38.1 0)
 			(show_name no)
@@
 			)
 		)
-		(property "Value" "Ra"
+		(property "Value" "5 kΩ"
 			(at 214.63 40.64 0)
 			(show_name no)
@@
 			(project "Michael_Samson_Onboarding"
 				(path "/e5003549-9df7-4e7c-9d3a-2812ef50da89"
-					(reference "R2")
+					(reference "RA1")
 					(unit 1)
 				)
@@
 			)
 		)
-		(property "Value" "C_Small_US"
-			(at 206.375 62.23 0)
+		(property "Value" "0.15 µF"
+			(at 210.82 62.23 0)
 			(show_name no)
 			(do_not_autoplace no)
@@
 		(in_pos_files yes)
 		(dnp no)
-		(property "Reference" "R1"
+		(property "Reference" "RB1"
 			(at 215.9 50.8 0)
 			(show_name no)
@@
 			)
 		)
-		(property "Value" "Ra"
-			(at 215.9 53.34 0)
+		(property "Value" "3 kΩ"
+			(at 214.63 53.34 0)
 			(show_name no)
 			(do_not_autoplace no)
@@
 			(project "Michael_Samson_Onboarding"
 				(path "/e5003549-9df7-4e7c-9d3a-2812ef50da89"
-					(reference "R1")
+					(reference "RB1")
 					(unit 1)
 				)
@@
 		(dnp no)
 		(fields_autoplaced yes)
-		(property "Reference" "R3"
-			(at 254.635 38.0999 0)
-			(show_name no)
-			(do_not_autoplace no)
-			(effects
-				(font
-					(size 1.27 1.27)
-				)
-				(justify left)
-			)
-		)
-		(property "Value" "R_Small_US"
-			(at 254.635 40.6399 0)
+		(property "Reference" "RL1"
+			(at 255.27 38.0999 0)
+			(show_name no)
+			(do_not_autoplace no)
+			(effects
+				(font
+					(size 1.27 1.27)
+				)
+				(justify left)
+			)
+		)
+		(property "Value" "1 kΩ"
+			(at 255.27 40.6399 0)
 			(show_name no)
 			(do_not_autoplace no)
@@
 			(project "Michael_Samson_Onboarding"
 				(path "/e5003549-9df7-4e7c-9d3a-2812ef50da89"
-					(reference "R3")
-					(unit 1)
-				)
+					(reference "RL1")
+					(unit 1)
+				)
