File: Onboarding/Franklin_Morgan_Onboarding/Franklin_Morgan_Onboarding.kicad_pcb (KiCad board)
At the start: 2 copper layers, 5 parts, among them J1 Conn_01x02_Pin, U1 NE555P

Commit message: PCB Update
Parts:
- C2: value 0.01u F -> 0.01uF
- moved C2 61.0 mm to (52.0, 89.0), turned to 90 degrees
- moved C1 54.2 mm to (59.0, 111.5), turned to 180 degrees
- moved J1 53.3 mm to (62.5, 90.5), turned to 180 degrees
- moved U1 46.5 mm to (53.8, 106.8), turned to 180 degrees
- moved RV1 35.4 mm to (66.5, 99.5)
Routing:
- net +5V: track 0.00 -> 45.7 mm, vias 0 -> 2
- net GND: track 0.00 -> 45.4 mm, vias 0 -> 2
- net Net-(U1-THRES): track 0.00 -> 30.4 mm
- net Net-(U1-DISCH): track 0.00 -> 21.2 mm, vias 0 -> 2
Other:
- board outline added: 47 x 33.5 mm
- board text added: "Franklin Morgan Servo Tester Onboarding"

Commit message: Added Thrust Stand Board
Routing:
- added copper zone on F.Cu, net GND
Changed lines of the file:
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@@
 		(net "Net-(U1-DISCH)")
+	)
+	(zone
+		(net "GND")
+		(layer "F.Cu")
+		(hatch edge 0.5)
+		(connect_pads
+			(clearance 0.5)
+		)
+		(min_thickness 0.25)
+		(fill yes
+			(thermal_gap 0.5)
+			(thermal_bridge_width 0.5)
+			(island_removal_mode 0)
+		)
+		(polygon
+			(pts
+				(xy 37 82.5) (xy 37 119) (xy 87.5 119) (xy 87 82.5)
+			)
+		)
 	)
 	(embedded_fonts no)
